Commit message: Oct14_1

File: install/fishbot_description/share/fishbot_description/urdf/fishbot_base.urdf (robot description, URDF)
Before this commit: robot fishbot, 2 links, 1 joints
Links:
- added link base_footprint
- added link caster_link, mass 0.02; collision sphere radius=0.016; visual sphere radius=0.016
- added link imu_link, mass 0.1; collision box size=0.02 0.02 0.02; visual box size=0.02 0.02 0.02
- added link left_wheel_link, mass 0.2; collision cylinder length=0.04 radius=0.032; visual cylinder length=0.04 radius=0.032
- added link right_wheel_link, mass 0.2; collision cylinder length=0.04 radius=0.032; visual cylinder length=0.04 radius=0.032
- link base_link: mass None -> 0.2; geometry collision cylinder length=0.12 radius=0.10; visual cylinder length=0.12 radius=0.10
- link laser_link: mass None -> 0.1; geometry collision cylinder length=0.02 radius=0.02; visual cylinder length=0.02 radius=0.02
Joints:
- added joint base_joint: type fixed, parent base_footprint, child base_link, origin xyz=0.0 0.0 0.076 rpy=0 0 0
- added joint caster_joint: type fixed, parent base_link, child caster_link, origin xyz=0.06 0.0 -0.076, axis 0 1 0
- added joint imu_joint: type fixed, parent base_link, child imu_link, origin xyz=0 0 0.02
- added joint left_wheel_joint: type continuous, parent base_link, child left_wheel_link, origin xyz=-0.02 0.10 -0.06, axis 0 1 0
- added joint right_wheel_joint: type continuous, parent base_link, child right_wheel_link, origin xyz=-0.02 -0.10 -0.06, axis 0 1 0
