Commit message: Nov13

File: install/fishbot_description/share/fishbot_description/urdf/fishbot_gazebo.urdf (robot description, URDF)
Before this commit: robot fishbot, 6 links, 5 joints
Links:
- added link imu_link, mass 0.1; collision box size=0.02 0.02 0.02; visual box size=0.02 0.02 0.02
Joints:
- added joint imu_joint: type fixed, parent base_link, child imu_link, origin xyz=0 0 0.02
